Commit message: Modified Bucket joint into revolute joint, also modified Passive wheels into spining wheels

File: src/mbot_gazebo/mbot/mbot_description/urdf/robotbody.xacro (robot description, xacro)
@@ -158,9 +158,15 @@
     </collision>
   </link>
-  <joint name="Joint_Bucket" type="fixed">
+  <joint name="Joint_Bucket" type="revolute">
     <origin xyz="0.35883098861838 0.2117 0.0476619772367585" rpy="0 0 0" />
     <parent link="base_link" />
     <child link="Bucket" />
-    <axis xyz="0 1 0" />
+    <axis xyz="0 1 0" /> <!-- If the rotation direction is opposite, change this "1" to "-1" -->
+    <limit
+    	lower="-0.5"
+    	upper="0.2"
+    	effort= "3"
+    	velocity="0.5"
+    />
   </joint>
 <!-- ************************** Camera ***********************-->

Commit message: Fixed the robot flying problem

File: src/mbot_gazebo/mbot/mbot_description/urdf/robotbody.xacro (robot description, xacro)
@@ -162,10 +162,10 @@
     <parent link="base_link" />
     <child link="Bucket" />
-    <axis xyz="0 1 0" /> <!-- If the rotation direction is opposite, change this "1" to "-1" -->
+    <axis xyz="0 -1 0" /> <!-- If the rotation direction is opposite, change this "1" to "-1" -->
     <limit
     	lower="-0.5"
     	upper="0.2"
-    	effort= "3"
-    	velocity="0.5"
+    	effort= "0.1"
+    	velocity="0.1"
     />
   </joint>
