Commit message: Fix robotbody configs_Try 1

File: src/mbot_gazebo/mbot/mbot_description/urdf/robotbody.gazebo.xacro (robot description, xacro)
@@ -13,5 +13,5 @@
 	<kp>10000000</kp>
 	<kd>1</kd>
-	<max_vel>0.5</max_vel>
+	<max_vel>0.7</max_vel>
   </gazebo>
   <gazebo reference="Left_Wheel">
@@ -21,5 +21,5 @@
 	<kp>10000000</kp>
 	<kd>1</kd>
-	<max_vel>0.5</max_vel>
+	<max_vel>0.7</max_vel>
   </gazebo>
   <gazebo reference="Bucket">
@@ -87,10 +87,10 @@
           <min>0.2</min>
           <max>12</max>
-          <resolution>0.005</resolution>
+          <resolution>0.015</resolution>
         </range>
         <noise>
-         <!-- <type>gaussian</type>
+          <type>gaussian</type>
           <mean>0.0</mean>
-          <stddev>0.00</stddev> -->
+          <stddev>0.01</stddev>
         </noise>
       </ray>
@@ -123,6 +123,6 @@
             <mean>0.0</mean>
             <stddev>1.7e-2</stddev>
-            <bias_mean>0.001</bias_mean>
-            <bias_stddev>0.00001</bias_stddev>
+            <bias_mean>0.1</bias_mean>
+            <bias_stddev>0.001</bias_stddev>
           </accel>
         </noise>
@@ -134,20 +134,20 @@
         <material>Gazebo/FlatBlack</material>
         <mu1>0</mu1>
-	<mu2>0</mu2>
+	<mu2>1</mu2>
   </gazebo>
   <gazebo reference="Right_Back_Wheel">
         <material>Gazebo/FlatBlack</material>
         <mu1>0</mu1>
-	<mu2>0</mu2>
+	<mu2>1</mu2>
   </gazebo>
   <gazebo reference="Left_Front_Wheel">
         <material>Gazebo/FlatBlack</material>
         <mu1>0</mu1>
-	<mu2>0</mu2>
+	<mu2>1</mu2>
   </gazebo>
   <gazebo reference="Left_Back_Wheel">
         <material>Gazebo/FlatBlack</material>
         <mu1>0</mu1>
-	<mu2>0</mu2>
+	<mu2>1</mu2>
   </gazebo>
   <gazebo>
@@ -156,7 +156,7 @@
     <leftJoint>Joint_Wheel_Left</leftJoint>
     <rightJoint>Joint_Wheel_Right</rightJoint>
-    <wheelSeparation>0.4898</wheelSeparation>
+    <wheelSeparation>0.45</wheelSeparation>
     <wheelDiameter>0.16</wheelDiameter>
-    <wheelAcceleration>1.5</wheelAcceleration>
+    <wheelAcceleration>2.0</wheelAcceleration>
     <wheelTorque>7</wheelTorque>
     <commandTopic>cmd_vel</commandTopic>

File: src/mbot_gazebo/mbot/mbot_description/urdf/robotbody.xacro (robot description, xacro)
@@ -12,5 +12,5 @@
     <inertial>
       <origin
-        xyz="0.249 0.00 0.3754" rpy="0 0 0" />
+        xyz="0.249258895595124 3.73456791304785E-17 0.375401162790698" rpy="0 0 0" />
        <mass value="1.35088484104347E-05" />
       <inertia
@@ -134,5 +134,5 @@
   <link name="Bucket">
     <inertial>
-      <origin xyz="-0.15184 -0.2117 0.041366" rpy="0 0 0" />
+      <origin xyz="-0.15184 -0.2117 0.07" rpy="0 0 0" />
       <mass value="20.752" />
       <inertia

Commit message: Change Wheel and dimension
Made some changes inside the robotbody.gazebo.xacro and robotbody.xacro files. Change the size of the wheels and frictions.

File: src/mbot_gazebo/mbot/mbot_description/urdf/robotbody.gazebo.xacro (robot description, xacro)
@@ -134,20 +134,20 @@
         <material>Gazebo/FlatBlack</material>
         <mu1>0</mu1>
-	<mu2>1</mu2>
+	      <mu2>0</mu2>
   </gazebo>
   <gazebo reference="Right_Back_Wheel">
         <material>Gazebo/FlatBlack</material>
         <mu1>0</mu1>
-	<mu2>1</mu2>
+	      <mu2>0</mu2>
   </gazebo>
   <gazebo reference="Left_Front_Wheel">
         <material>Gazebo/FlatBlack</material>
         <mu1>0</mu1>
-	<mu2>1</mu2>
+	      <mu2>0</mu2>
   </gazebo>
   <gazebo reference="Left_Back_Wheel">
         <material>Gazebo/FlatBlack</material>
         <mu1>0</mu1>
-	<mu2>1</mu2>
+	      <mu2></mu2>
   </gazebo>
   <gazebo>
@@ -157,7 +157,7 @@
     <rightJoint>Joint_Wheel_Right</rightJoint>
     <wheelSeparation>0.45</wheelSeparation>
-    <wheelDiameter>0.16</wheelDiameter>
+    <wheelDiameter>0.12</wheelDiameter>
     <wheelAcceleration>2.0</wheelAcceleration>
-    <wheelTorque>7</wheelTorque>
+    <wheelTorque>10</wheelTorque>
     <commandTopic>cmd_vel</commandTopic>
     <odometryTopic>odom</odometryTopic>

File: src/mbot_gazebo/mbot/mbot_description/urdf/robotbody.xacro (robot description, xacro)
@@ -237,5 +237,5 @@
     <inertial>
       <origin  xyz="-0.016839 0.2459 0.041366" rpy="0 0 0" />
-      <mass value="2.752" />
+      <mass value="2" />
       <inertia
         ixx="0"
@@ -260,5 +260,5 @@
     </collision>
   </link>
-  <joint name="Joint_Wheel_Front_Right" type="continuous">
+  <joint name="Joint_Wheel_Front_Right"  type="continuous">
     <origin xyz="0.22383 -0.2459 0.047662" rpy="0 0 0" />
     <parent link="base_link" />
@@ -269,5 +269,5 @@
     <inertial>
       <origin xyz="0.46316 0.246 0.041366" rpy="0 0 0" />
-      <mass value="2.752" />
+      <mass value="2" />
       <inertia
         ixx="0"
@@ -292,5 +292,5 @@
     </collision>
   </link>
-  <joint name="Joint_Wheel_Back_Right" type="continuous">
+  <joint name="Joint_Wheel_Back_Right"  type="continuous">
     <origin xyz="-0.25617 -0.246 0.047662" rpy="0 0 0" />
     <parent link="base_link" />
@@ -301,5 +301,5 @@
     <inertial>
       <origin xyz="-0.016839 -0.2459 0.041366" rpy="0 0 0" />
-      <mass value="2.752" />
+      <mass value="2" />
       <inertia
         ixx="0"
@@ -324,5 +324,5 @@
     </collision>
   </link>
-  <joint name="Joint_Wheel_Front_Left" type="continuous">
+  <joint name="Joint_Wheel_Front_Left"  type="continuous">
     <origin xyz="0.22383 0.2459 0.047662" rpy="0 0 0" />
     <parent link="base_link" />
@@ -333,5 +333,5 @@
     <inertial>
       <origin xyz="0.46316 -0.2459 0.041366" rpy="0 0 0" />
-      <mass value="2.752" />
+      <mass value="2" />
       <inertia
         ixx="0"
@@ -356,5 +356,5 @@
     </collision>
   </link>
-  <joint name="Joint_Wheel_Back_Left" type="continuous">
+  <joint name="Joint_Wheel_Back_Left"  type="continuous">
     <origin xyz="-0.25617 0.2459 0.047662" rpy="0 0 0" />
     <parent link="base_link" />

Commit message: fixed bugs wheel size

File: src/mbot_gazebo/mbot/mbot_description/urdf/robotbody.gazebo.xacro (robot description, xacro)
@@ -134,20 +134,20 @@
         <material>Gazebo/FlatBlack</material>
         <mu1>0</mu1>
-	      <mu2>0</mu2>
+	<mu2>0</mu2>
   </gazebo>
   <gazebo reference="Right_Back_Wheel">
         <material>Gazebo/FlatBlack</material>
         <mu1>0</mu1>
-	      <mu2>0</mu2>
+	<mu2>0</mu2>
   </gazebo>
   <gazebo reference="Left_Front_Wheel">
         <material>Gazebo/FlatBlack</material>
         <mu1>0</mu1>
-	      <mu2>0</mu2>
+	<mu2>0</mu2>
   </gazebo>
   <gazebo reference="Left_Back_Wheel">
         <material>Gazebo/FlatBlack</material>
         <mu1>0</mu1>
-	      <mu2></mu2>
+	<mu2>0</mu2>
   </gazebo>
   <gazebo>
@@ -159,5 +159,5 @@
     <wheelDiameter>0.12</wheelDiameter>
     <wheelAcceleration>2.0</wheelAcceleration>
-    <wheelTorque>10</wheelTorque>
+    <wheelTorque>7</wheelTorque>
     <commandTopic>cmd_vel</commandTopic>
     <odometryTopic>odom</odometryTopic>

File: src/mbot_gazebo/mbot/mbot_description/urdf/robotbody.xacro (robot description, xacro)
@@ -260,5 +260,5 @@
     </collision>
   </link>
-  <joint name="Joint_Wheel_Front_Right"  type="continuous">
+  <joint name="Joint_Wheel_Front_Right" type="continuous">
     <origin xyz="0.22383 -0.2459 0.047662" rpy="0 0 0" />
     <parent link="base_link" />
@@ -292,5 +292,5 @@
     </collision>
   </link>
-  <joint name="Joint_Wheel_Back_Right"  type="continuous">
+  <joint name="Joint_Wheel_Back_Right" type="continuous">
     <origin xyz="-0.25617 -0.246 0.047662" rpy="0 0 0" />
     <parent link="base_link" />
@@ -324,5 +324,5 @@
     </collision>
   </link>
-  <joint name="Joint_Wheel_Front_Left"  type="continuous">
+  <joint name="Joint_Wheel_Front_Left" type="continuous">
     <origin xyz="0.22383 0.2459 0.047662" rpy="0 0 0" />
     <parent link="base_link" />
@@ -356,5 +356,5 @@
     </collision>
   </link>
-  <joint name="Joint_Wheel_Back_Left"  type="continuous">
+  <joint name="Joint_Wheel_Back_Left" type="continuous">
     <origin xyz="-0.25617 0.2459 0.047662" rpy="0 0 0" />
     <parent link="base_link" />

Commit message: adding communication protocol to STM

File: src/mbot_gazebo/mbot/mbot_description/urdf/robotbody.gazebo.xacro (robot description, xacro)
@@ -133,21 +133,21 @@
   <gazebo reference="Right_Front_Wheel">
         <material>Gazebo/FlatBlack</material>
-        <mu1>0.001</mu1>
-	<mu2>0.001</mu2>
+        <mu1>0.05</mu1>
+	<mu2>0.05</mu2>
   </gazebo>
   <gazebo reference="Right_Back_Wheel">
         <material>Gazebo/FlatBlack</material>
-        <mu1>0.001</mu1>
-	<mu2>0.001</mu2>
+        <mu1>0.05</mu1>
+	<mu2>0.05</mu2>
   </gazebo>
   <gazebo reference="Left_Front_Wheel">
         <material>Gazebo/FlatBlack</material>
-        <mu1>0.001</mu1>
-	<mu2>0.001</mu2>
+        <mu1>0.05</mu1>
+	<mu2>0.05</mu2>
   </gazebo>
   <gazebo reference="Left_Back_Wheel">
         <material>Gazebo/FlatBlack</material>
-        <mu1>0.001</mu1>
-	<mu2>0.001</mu2>
+        <mu1>0.05</mu1>
+	<mu2>0.05</mu2>
   </gazebo>
   <gazebo>

File: src/mbot_gazebo/mbot/mbot_description/urdf/robotbody.xacro (robot description, xacro)
@@ -158,15 +158,9 @@
     </collision>
   </link>
-  <joint name="Joint_Bucket" type="revolute">
+  <joint name="Joint_Bucket" type="fixed">
     <origin xyz="0.35883098861838 0.2117 0.0476619772367585" rpy="0 0 0" />
     <parent link="base_link" />
     <child link="Bucket" />
-    <axis xyz="0 -1 0" /> <!-- If the rotation direction is opposite, change this "1" to "-1" -->
-    <limit
-    	lower="-0.5"
-    	upper="0.2"
-    	effort= "0.1"
-    	velocity="0.1"
-    />
+    <axis xyz="0 1 0" />
   </joint>
 <!-- ************************** Camera ***********************-->
