Commit message: Add files via upload

File: src/ugv_description/urdf/ugv.urdf (robot description, URDF)
Before this commit: robot UGV_Unimelb, 10 links, 9 joints
Links:
- link Bucket: mass 15 -> 1
- link Lidar_link: mass 4 -> 1
- link left_back_wheel: mass 5 -> 1
- link left_front_wheel: mass 5 -> 1
- link left_wheel: mass 5 -> 1
- link right_back_wheel: mass 5 -> 1
- link right_front_wheel: mass 5 -> 1
- link right_wheel: mass 5 -> 1
- link robot_body: mass 25 -> 5
Joints:
- removed joint Joint_Camera
- removed joint Joint_Lidar
- added joint joint_camera: type fixed, parent robot_body, child Camera_link, origin xyz=0.29633 0 0.337 rpy=0 0 0, axis 0 0 0
- added joint joint_lidar: type continuous, parent robot_body, child Lidar_link, origin xyz=0.21533 0 0.403 rpy=0 0 0, axis 0 0 1
